File: NANOLNA.kicad_sch (KiCad schematic)
At the start: 12 parts, among them J1 Conn_Coaxial, J2 USB_C_Receptacle_PowerOnly_6P, J3 Conn_Coaxial, J4 JST MOUNT, U1 PMA3-83LN_

Commit message: made it nano-er
Parts:
- renumbered J2 to J1, J1 to J2, J4 to J3, J3 to J4
Changed lines of the file:
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@@
 		(on_board yes)
 		(dnp no)
-		(property "Reference" "J2"
+		(property "Reference" "J1"
 			(at 34.29 16.256 0)
 			(effects
@@
 			(project "random rf stuff"
 				(path "/32a38c29-f6c2-4b2a-9669-d7bdc565a805"
-					(reference "J2")
+					(reference "J1")
 					(unit 1)
 				)
@@
 		(dnp no)
 		(fields_autoplaced yes)
-		(property "Reference" "#PWR03"
+		(property "Reference" "#PWR0107"
 			(at 49.53 85.09 0)
 			(effects
@@
 			(project "random rf stuff"
 				(path "/32a38c29-f6c2-4b2a-9669-d7bdc565a805"
-					(reference "#PWR03")
+					(reference "#PWR0107")
 					(unit 1)
 				)
@@
 		(on_board yes)
 		(dnp no)
-		(property "Reference" "J4"
+		(property "Reference" "J3"
 			(at 91.694 51.816 0)
 			(effects
@@
 			(project "random rf stuff"
 				(path "/32a38c29-f6c2-4b2a-9669-d7bdc565a805"
-					(reference "J4")
+					(reference "J3")
 					(unit 1)
 				)
@@
 		(dnp no)
 		(fields_autoplaced yes)
-		(property "Reference" "J3"
+		(property "Reference" "J4"
 			(at 110.49 72.6831 0)
 			(effects
@@
 			(project "random rf stuff"
 				(path "/32a38c29-f6c2-4b2a-9669-d7bdc565a805"
-					(reference "J3")
+					(reference "J4")
 					(unit 1)
 				)
@@
 		(on_board yes)
 		(dnp no)
-		(property "Reference" "#PWR04"
+		(property "Reference" "#PWR0102"
 			(at 63.5 64.77 0)
 			(effects
@@
 			(project "random rf stuff"
 				(path "/32a38c29-f6c2-4b2a-9669-d7bdc565a805"
-					(reference "#PWR04")
+					(reference "#PWR0102")
 					(unit 1)
 				)
@@
 		(on_board yes)
 		(dnp no)
-		(property "Reference" "#PWR06"
+		(property "Reference" "#PWR0101"
 			(at 73.66 64.77 0)
 			(effects
@@
 			(project "random rf stuff"
 				(path "/32a38c29-f6c2-4b2a-9669-d7bdc565a805"
-					(reference "#PWR06")
+					(reference "#PWR0101")
 					(unit 1)
 				)
@@
 		(on_board yes)
 		(dnp no)
-		(property "Reference" "#PWR09"
+		(property "Reference" "#PWR0104"
 			(at 96.52 53.34 0)
 			(effects
@@
 			(project "random rf stuff"
 				(path "/32a38c29-f6c2-4b2a-9669-d7bdc565a805"
-					(reference "#PWR09")
+					(reference "#PWR0104")
 					(unit 1)
 				)
@@
 		(dnp no)
 		(fields_autoplaced yes)
-		(property "Reference" "#PWR07"
+		(property "Reference" "#PWR0103"
 			(at 73.66 87.63 0)
 			(effects
@@
 			(project "random rf stuff"
 				(path "/32a38c29-f6c2-4b2a-9669-d7bdc565a805"
-					(reference "#PWR07")
+					(reference "#PWR0103")
 					(unit 1)
 				)
@@
 		(dnp no)
 		(fields_autoplaced yes)
-		(property "Reference" "#PWR02"
+		(property "Reference" "#PWR0106"
 			(at 30.48 55.88 0)
 			(effects
@@
 			(project "random rf stuff"
 				(path "/32a38c29-f6c2-4b2a-9669-d7bdc565a805"
-					(reference "#PWR02")
+					(reference "#PWR0106")
 					(unit 1)
 				)
@@
 		(on_board yes)
 		(dnp no)
-		(property "Reference" "#PWR01"
+		(property "Reference" "#PWR0109"
 			(at 36.83 74.93 0)
 			(effects
@@
 			(project "random rf stuff"
 				(path "/32a38c29-f6c2-4b2a-9669-d7bdc565a805"
-					(reference "#PWR01")
+					(reference "#PWR0109")
 					(unit 1)
 				)
@@
 		(on_board yes)
 		(dnp no)
-		(property "Reference" "#PWR05"
+		(property "Reference" "#PWR0108"
 			(at 57.15 44.45 0)
 			(effects
@@
 			(project "random rf stuff"
 				(path "/32a38c29-f6c2-4b2a-9669-d7bdc565a805"
-					(reference "#PWR05")
+					(reference "#PWR0108")
 					(unit 1)
 				)
@@
 		(on_board yes)
 		(dnp no)
-		(property "Reference" "#PWR08"
+		(property "Reference" "#PWR0105"
 			(at 106.68 85.09 0)
 			(effects
@@
 			(project "random rf stuff"
 				(path "/32a38c29-f6c2-4b2a-9669-d7bdc565a805"
-					(reference "#PWR08")
+					(reference "#PWR0105")
 					(unit 1)
 				)
@@
 		(on_board yes)
 		(dnp no)
-		(property "Reference" "J1"
+		(property "Reference" "J2"
 			(at 40.64 76.454 0)
 			(effects
@@
 			(project "random rf stuff"
 				(path "/32a38c29-f6c2-4b2a-9669-d7bdc565a805"
-					(reference "J1")
-					(unit 1)
-				)
+					(reference "J2")
+					(unit 1)
+				)
